File: Stage1 - STM/voxboard/voxboard.kicad_sch (KiCad schematic)
At the start: 174 parts, among them IC1 TPS54331DR, J1 USB4110-GF-A, J11 Conn_01x04_Pin, J12 Conn_01x04_Pin, J13 Conn_01x04_Pin, J14 Conn_01x04_Pin, J15 Conn_01x04_Pin, J16 Conn_01x04_Pin, J17 Conn_01x04_Pin, J18 Conn_01x04_Pin, Q1 PMOS, Q2 PMOS, SW2 SW_Push, SW3 SW_SPDT, U1 STM32F446RETx, U11 SN65HVD230DR, U12 TPD4E02B04DQAR, U14 PESD5V0F1BRSFYL, U15 PESD5V0F1BRSFYL, U16 SM12OC, U18 MT6835, U19 MT6835, U2 AP7361C-33Y5-13, U20 MT6835, U21 MT6835, U22 MT6835, U3 TPD4E02B04DQAR, U4 SM12OC, U5 TPD2E1B06DRLR, U6 MT6835, Y1 8MHz

Commit message: Updated JOURNAL.md
Parts:
- removed C49, C50: 100n, Capacitor_SMD:C_0402_1005Metric, symbol Device:C
- removed C51: 100u, Capacitor_THT:CP_Radial_D8.0mm_P3.50mm, symbol Device:C_Polarized
- removed DRIVER4: TMC2209, Arsenal_Lib:MODULE_TMC2209_5160, symbol Arsenal_Lib:TMC2209
- removed JM4: Conn_01x04_Pin, Arsenal_Lib:JST_VH_B4P-VH-FB-B_1x04_P3.96mm_Vertical, symbol Connector:Conn_01x04_Pin
- removed R17: 33o, Resistor_SMD:R_0402_1005Metric, symbol Device:R
- removed R28: 10k, Resistor_SMD:R_0402_1005Metric, symbol Device:R
- added C53: 100u, Capacitor_THT:CP_Radial_D8.0mm_P3.50mm, symbol Device:C_Polarized
- added C54: 1u, Capacitor_SMD:C_0603_1608Metric, symbol Device:C
- added C55, C56: 100n, Capacitor_SMD:C_0402_1005Metric, symbol Device:C
- added C57: 220u, Capacitor_THT:CP_Radial_D10.0mm_P5.00mm, symbol Device:C_Polarized
- added DRIVER6: TMC5160, Arsenal_Lib:MODULE_TMC2209_5160, symbol Arsenal_Lib:TMC5160
- added JM6: Conn_01x04_Pin, Arsenal_Lib:JST_VH_B4P-VH-FB-B_1x04_P3.96mm_Vertical, symbol Connector:Conn_01x04_Pin
- added R54, R56: 10k, Resistor_SMD:R_0402_1005Metric, symbol Device:R
- added R55: 33o, Resistor_SMD:R_0402_1005Metric, symbol Device:R
- R19: value 1k -> 33o
- renumbered DRIVER5 to DRIVER4, DRIVER6 to DRIVER5, JM5 to JM4, JM6 to JM5
Connections:
- net +24V: now also C53.1, C54.2, C56.1, C57.1, DRIVER6.8 (VM)
- net +3.3V: now also DRIVER3.14 (MS2), C55.1, DRIVER6.2 (VDD), R54.2, R56.2
- net GND: now also C53.2, C54.1, C55.2, C56.2, C57.2, DRIVER6.1 (GND), DRIVER6.11 (CLK), DRIVER6.7 (GND); no longer DRIVER3.14 (MS2)
- net SPI1_MISO: now also DRIVER6.12 (SDO)
- net SPI1_MOSI: now also DRIVER6.15 (SDI)
- net SPI1_SCK: now also DRIVER6.14 (SCK)
- net UARTTX_MOT_U1: no longer DRIVER1.12 (PDN/UART), DRIVER2.12 (PDN/UART), R18.1
- net UARTTX_MOT_U2: no longer DRIVER3.12 (PDN/UART), R19.1
- net at R19.2: now also DRIVER6.10 (STEP); no longer U1.16 (PA2)
- net at R16.2: now also U1.16 (PA2)
- net DIAG_MOT_U1_00 renamed DIAG_MOT_SPI_10
- net DIAG_MOT_SPI_10: now also DRIVER6.17 (DIAG0), R56.1; no longer DRIVER1.18 (DIAG)
- net DIAG_MOT_U1_01 renamed DIAG_MOT_U_01
- net DIAG_MOT_U2_00 renamed DIAG_MOT_U_10
- net DIR_MOT_U1_00 renamed DIR_MOT_U_00
- net DIR_MOT_U1_01 renamed DIR_MOT_U_01
- net DIR_MOT_U2_00 renamed DIR_MOT_U_10
- net DIR_MOT_U2_01 renamed DIR_MOT_SPI_10
- net DIR_MOT_SPI_10: now also R55.1
- net EN_MOT_U1_00 renamed EN_MOT_U_00
- net EN_MOT_U1_01 renamed EN_MOT_U_01
- net EN_MOT_U2_00 renamed EN_MOT_U_10
- net EN_MOT_U2_01 renamed EN_MOT_SPI_10
- net EN_MOT_SPI_10: now also DRIVER6.16 (~{EN}), R54.1
- net STEP_MOT_U1_00 renamed STEP_MOT_U_00
- net STEP_MOT_U1_01 renamed STEP_MOT_U_01
- net STEP_MOT_U2_00 renamed STEP_MOT_U_10
- net STEP_MOT_U2_01 renamed CS_MOT_SPI_10
- net CS_MOT_SPI_10: now also DRIVER6.13 (CSN); no longer U1.58 (PB6)
- new net: DRIVER6.9 (DIR), R55.2
- new net: DRIVER6.4 (B2), JM6.1 (Pin_1)
- new net: DRIVER6.5 (A1), JM6.2 (Pin_2)
- new net: DRIVER6.3 (B1), JM6.3 (Pin_3)
- new net: DRIVER6.6 (A2), JM6.4 (Pin_4)
- new net DIAG_MOT_U_00: DRIVER1.18 (DIAG)
- new net STEP_MOT_SPI_10: R19.1, U1.58 (PB6)
- new net UARTTX_MOT: DRIVER1.12 (PDN/UART), DRIVER2.12 (PDN/UART), DRIVER3.12 (PDN/UART), R18.1
- no-connect marks 26 -> 23
Other:
- note added: "ESD USBC"
- note added: "TMC2209 : USART1 : ADDRESS - 10"
- note added: "TMC5160 : SPI1 : USER_ADDRESS - 10"
- note removed: "ESD USBLC6-2SC6"
- note removed: "TMC2209 : USART2 : ADDRESS - 00"
- note removed: "TMC2209 : USART2 : ADDRESS - 01"
- moved on the sheet: C10, C23, C24, C26, C37, C38, C39, C52, C7, D1, D4, DRIVER4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

Commit message: Updated JOURNAL.md
Parts:
- removed U15: PESD5V0F1BRSFYL, Diode_SMD:Nexperia_DSN0603-2_0.6x0.3mm_P0.4mm, symbol Arsenal_Lib:PESD5V0F1BRSFYL
Connections:
- net UARTTX_MOT_U1 is gone; now on net UARTTX_MOT: U14.1
Other:
- moved on the sheet: D7, JS1, JU1, R26, R30, R31, R52, SW3, U4
