File: Stage1 - STM/voxboard/voxboard.kicad_sch (KiCad schematic)
At the start: 179 parts, among them IC1 TPS54331DR, J1 USB4110-GF-A, J11 Conn_01x04_Pin, J12 Conn_01x04_Pin, J13 Conn_01x04_Pin, J14 Conn_01x04_Pin, J15 Conn_01x04_Pin, J16 Conn_01x04_Pin, J17 Conn_01x04_Pin, J18 Conn_01x04_Pin, Q1 PMOS, Q2 PMOS, SW2 SW_Push, SW3 SW_SPDT, U1 STM32F446RETx, U11 SN65HVD230DR, U12 TPD4E02B04DQAR, U14 PESD5V0F1BRSFYL, U16 SM12OC, U18 MT6835, U19 MT6835, U2 AP7361C-33Y5-13, U20 MT6835, U21 MT6835, U22 MT6835, U3 TPD4E02B04DQAR, U4 SM12OC, U5 TPD2E1B06DRLR, U6 MT6835, Y1 8MHz

Commit message: Updates
Parts:
- C24: footprint Capacitor_THT:CP_Radial_D8.0mm_P3.50mm -> Capacitor_THT:CP_Radial_D12.5mm_P5.00mm
- C25, C29, C58, C7: footprint Capacitor_SMD:C_0603_1608Metric -> Capacitor_SMD:C_0805_2012Metric
- C53: footprint Capacitor_THT:CP_Radial_D8.0mm_P3.50mm -> Capacitor_THT:CP_Radial_D6.3mm_P2.50mm
- D2: footprint Diode_SMD:D_SMA -> Diode_SMD:D_SMC
- D8: footprint Diode_SMD:D_SMC -> Package_TO_SOT_SMD:SOT-23
- R2: footprint Resistor_SMD:R_0402_1005Metric -> Resistor_SMD:R_0603_1608Metric
Other:
- moved on the sheet: TP1
Changed lines of the file:
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@@
 	(wire
 		(pts
+			(xy 157.48 41.91) (xy 158.75 41.91)
+		)
+		(stroke
+			(width 0)
+			(type default)
+		)
+	)
+	(wire
+		(pts
 			(xy 358.14 205.74) (xy 372.11 205.74)
 		)
@@
 			)
 		)
-		(property "Footprint" "Capacitor_THT:CP_Radial_D8.0mm_P3.50mm"
+		(property "Footprint" "Capacitor_THT:CP_Radial_D12.5mm_P5.00mm"
 			(at 56.1848 31.75 0)
 			(effects
@@
 			)
 		)
-		(property "Footprint" "Capacitor_SMD:C_0603_1608Metric"
+		(property "Footprint" "Capacitor_SMD:C_0805_2012Metric"
 			(at 191.4652 72.39 0)
 			(effects
@@
 			)
 		)
-		(property "Footprint" "Capacitor_SMD:C_0603_1608Metric"
+		(property "Footprint" "Capacitor_SMD:C_0805_2012Metric"
 			(at 70.8152 39.37 0)
 			(effects
@@
 			)
 		)
-		(property "Footprint" "Capacitor_THT:CP_Radial_D8.0mm_P3.50mm"
+		(property "Footprint" "Capacitor_THT:CP_Radial_D6.3mm_P2.50mm"
 			(at 62.5348 31.75 0)
 			(effects
@@
 			)
 		)
-		(property "Footprint" "Capacitor_SMD:C_0603_1608Metric"
+		(property "Footprint" "Capacitor_SMD:C_0805_2012Metric"
 			(at 23.1648 223.52 0)
 			(effects
@@
 			)
 		)
-		(property "Footprint" "Diode_SMD:D_SMC"
+		(property "Footprint" "Package_TO_SOT_SMD:SOT-23"
 			(at 220.98 33.02 0)
 			(effects
@@
 			)
 		)
-		(property "Footprint" "Capacitor_SMD:C_0603_1608Metric"
+		(property "Footprint" "Capacitor_SMD:C_0805_2012Metric"
 			(at 41.6052 52.07 0)
 			(effects
@@
 			)
 		)
-		(property "Footprint" "Resistor_SMD:R_0402_1005Metric"
+		(property "Footprint" "Resistor_SMD:R_0603_1608Metric"
 			(at 123.698 38.1 90)
 			(effects
@@
 	(symbol
 		(lib_id "Connector:TestPoint")
-		(at 158.75 41.91 90)
+		(at 157.48 41.91 90)
 		(mirror x)
 		(unit 1)
@@
 		(dnp no)
 		(property "Reference" "TP1"
-			(at 157.48 43.942 90)
+			(at 156.21 43.942 90)
 			(effects
 				(font
@@
 		)
 		(property "Value" "TestPoint"
-			(at 153.67 43.1799 90)
+			(at 152.4 43.1799 90)
 			(effects
 				(font
@@
 		)
 		(property "Footprint" "TestPoint:TestPoint_Pad_2.0x2.0mm"
-			(at 158.75 46.99 0)
+			(at 157.48 46.99 0)
 			(effects
 				(font
@@
 		)
 		(property "Datasheet" "~"
-			(at 158.75 46.99 0)
+			(at 157.48 46.99 0)
 			(effects
 				(font
@@
 		)
 		(property "Description" "test point"
-			(at 158.75 41.91 0)
+			(at 157.48 41.91 0)
 			(effects
 				(font
@@
 			)
 		)
-		(property "Footprint" "Diode_SMD:D_SMA"
+		(property "Footprint" "Diode_SMD:D_SMC"
 			(at 168.91 35.56 0)
 			(effects
