File: Stage1 - STM/voxboard/voxboard.kicad_pcb (KiCad board)
At the start: 4 copper layers, 174 parts, among them IC1 TPS54331DR, J1 USB4110-GF-A, J11 Conn_01x04_Pin, J12 Conn_01x04_Pin, J13 Conn_01x04_Pin, J14 Conn_01x04_Pin, J15 Conn_01x04_Pin, J16 Conn_01x04_Pin, J17 Conn_01x04_Pin, J18 Conn_01x04_Pin, Q1 PMOS, Q2 PMOS, SW2 SW_Push, SW3 SW_SPDT, U1 STM32F446RETx, U11 SN65HVD230DR, U12 TPD4E02B04DQAR, U14 PESD5V0F1BRSFYL, U15 PESD5V0F1BRSFYL, U16 SM12OC, U18 MT6835, U19 MT6835, U2 AP7361C-33Y5-13, U20 MT6835, U21 MT6835, U22 MT6835, U3 TPD4E02B04DQAR, U4 SM12OC, U5 TPD2E1B06DRLR, U6 MT6835, Y1 8MHz

Commit message: Updated JOURNAL.md
Parts:
- removed C49, C50: 100n, Capacitor_SMD:C_0402_1005Metric
- removed C51: 100u, Capacitor_THT:CP_Radial_D8.0mm_P3.50mm
- removed the DRIVER4 at (226.9, 91.9)
- removed the JM4 at (242.6, 85.9)
- removed R16, R17: 33o, Resistor_SMD:R_0402_1005Metric
- removed R28: 10k, Resistor_SMD:R_0402_1005Metric
- added C53: 100u, Capacitor_THT:CP_Radial_D8.0mm_P3.50mm, F.Cu at (191.9, 161.8)
- added C54: 1u, Capacitor_SMD:C_0603_1608Metric, F.Cu at (196.8, 161.8)
- added C55: 100n, Capacitor_SMD:C_0402_1005Metric, F.Cu at (229.6, 90.2)
- added C56: 100n, Capacitor_SMD:C_0402_1005Metric, F.Cu at (229.6, 92.2)
- added C57: 220u, Capacitor_THT:CP_Radial_D10.0mm_P5.00mm, F.Cu at (211.8, 102.9)
- added DRIVER6: TMC5160, Arsenal_Lib:MODULE_TMC2209_5160, F.Cu at (227.2, 92.2)
- added JM6: Conn_01x04_Pin, Arsenal_Lib:JST_VH_B4P-VH-FB-B_1x04_P3.96mm_Vertical, F.Cu at (243.0, 86.1)
- added R19: 33o, Resistor_SMD:R_0402_1005Metric, F.Cu at (226.7, 90.3)
- added R54: 10k, Resistor_SMD:R_0402_1005Metric, F.Cu at (226.7, 92.2)
- added R55: 33o, Resistor_SMD:R_0402_1005Metric, F.Cu at (226.7, 94.2)
- added R56: 10k, Resistor_SMD:R_0402_1005Metric, F.Cu at (226.7, 96.2)
- moved PS1 3.72 mm to (212.8, 145.6)
- renumbered DRIVER5 to DRIVER4, DRIVER6 to DRIVER5, JM5 to JM4, JM6 to JM5
Connections:
- net DIAG_MOT_U1_01 renamed DIAG_MOT_U_01
- net DIAG_MOT_U2_00 renamed DIAG_MOT_U_10
- net DIR_MOT_U1_00 renamed DIR_MOT_U_00
- net DIR_MOT_U1_01 renamed DIR_MOT_U_01
- net DIR_MOT_U2_00 renamed DIR_MOT_U_10
- net EN_MOT_U1_00 renamed EN_MOT_U_00
- net EN_MOT_U1_01 renamed EN_MOT_U_01
- net EN_MOT_U2_00 renamed EN_MOT_U_10
- net STEP_MOT_U1_00 renamed STEP_MOT_U_00
- net STEP_MOT_U1_01 renamed STEP_MOT_U_01
- net STEP_MOT_U2_00 renamed STEP_MOT_U_10
- DRIVER1 pad 12: UARTTX_MOT_U1 -> UARTTX_MOT
- DRIVER1 pad 18: DIAG_MOT_U1_00 -> DIAG_MOT_U_00
- DRIVER2 pad 12: UARTTX_MOT_U1 -> UARTTX_MOT
- DRIVER3 pad 12: UARTTX_MOT_U2 -> UARTTX_MOT
- DRIVER3 pad 14: GND -> VMCU
- R18 pad 1: UARTTX_MOT_U1 -> UARTTX_MOT
- U1 pad 11: DIR_MOT_U2_01 -> DIR_MOT_SPI_10
- U1 pad 16: Net-(U1-PA2) -> CS_MOT_SPI_10
- U1 pad 43: EN_MOT_U2_01 -> EN_MOT_SPI_10
- U1 pad 54: DIAG_MOT_U1_00 -> DIAG_MOT_SPI_10
- U1 pad 58: STEP_MOT_U2_01 -> STEP_MOT_SPI_10

Commit message: Bulk
Parts:
- removed FB1: 600R, Inductor_SMD:L_1210_3225Metric
- removed the R19 at (144.2, 89.0)
- removed U15: PESD5V0F1BRSFYL, Diode_SMD:Nexperia_DSN0603-2_0.6x0.3mm_P0.4mm
- added C49: 100n, Capacitor_SMD:C_0402_1005Metric, F.Cu at (168.3, 54.8)
- added C50: 1u, Capacitor_SMD:C_0603_1608Metric, F.Cu at (168.2, 51.8)
- added C51: 22u, Capacitor_THT:CP_Radial_D5.0mm_P2.00mm, F.Cu at (167.3, 48.2)
- added C58: 10u, Capacitor_SMD:C_0603_1608Metric, F.Cu at (168.2, 53.4)
- added G***: LOGO, LOGO, F.Cu at (159.3, 49.1)
- added G***: LOGO, LOGO, B.Cu at (129.2, 39.8)
- added G***: LOGO, LOGO, B.Cu at (129.4, 57.3)
- added R16: 33o, Resistor_SMD:R_0402_1005Metric, F.Cu at (130.7, 39.1)
- JM1, JM2, JM3, JM4, JM5, JM6: footprint Arsenal_Lib:JST_VH_B4P-VH-FB-B_1x04_P3.96mm_Vertical -> Connector_JST:JST_XA_B04B-XASK-1_1x04_P2.50mm_Vertical
- moved C26 201.0 mm to (77.3, 83.0), turned to 180 degrees
- moved R39 198.5 mm to (75.8, 76.1), turned to 90 degrees
- moved R37 195.4 mm to (78.3, 76.1), turned to 90 degrees
- moved C39 190.4 mm to (98.2, 85.8), turned to 0 degrees
- moved DRIVER4 189.4 mm to (84.7, 79.3), turned to 90 degrees
- moved C37 183.8 mm to (92.3, 83.8), turned to 180 degrees
- moved R38 182.0 mm to (88.5, 75.2), turned to 90 degrees
- moved R49 181.0 mm to (91.2, 77.4), turned to 90 degrees
- moved JM5 170.5 mm to (95.7, 21.7), turned to 0 degrees
- moved JM4 168.5 mm to (88.7, 93.4), turned to 180 degrees
- moved C46 165.7 mm to (109.8, 83.3), turned to 180 degrees
- moved R48 163.8 mm to (92.9, 37.5), turned to 90 degrees
- moved R34 163.7 mm to (94.1, 39.0), turned to 90 degrees
- moved R10 161.8 mm to (108.6, 75.4), turned to 90 degrees
- moved R9 159.2 mm to (110.9, 75.4), turned to 90 degrees
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Connections:
- JM1 pad 1: Net-(DRIVER1-B1) -> Net-(DRIVER1-A1)
- JM1 pad 2: Net-(DRIVER1-A1) -> Net-(DRIVER1-B1)
- JM2 pad 1: Net-(DRIVER2-B1) -> Net-(DRIVER2-A1)
- JM2 pad 2: Net-(DRIVER2-A1) -> Net-(DRIVER2-B1)
- JM3 pad 1: Net-(DRIVER3-B1) -> Net-(DRIVER3-A1)
- JM3 pad 2: Net-(DRIVER3-A1) -> Net-(DRIVER3-B1)
- JM4 pad 1: Net-(DRIVER4-B2) -> Net-(DRIVER4-A1)
- JM4 pad 2: Net-(DRIVER4-A1) -> Net-(DRIVER4-B1)
- JM4 pad 3: Net-(DRIVER4-B1) -> Net-(DRIVER4-A2)
- JM4 pad 4: Net-(DRIVER4-A2) -> Net-(DRIVER4-B2)
- JM5 pad 1: Net-(DRIVER5-B2) -> Net-(DRIVER5-A1)
- JM5 pad 2: Net-(DRIVER5-A1) -> Net-(DRIVER5-B1)
- JM5 pad 3: Net-(DRIVER5-B1) -> Net-(DRIVER5-A2)
- JM5 pad 4: Net-(DRIVER5-A2) -> Net-(DRIVER5-B2)
- JM6 pad 1: Net-(DRIVER6-B2) -> Net-(DRIVER6-A1)
- JM6 pad 2: Net-(DRIVER6-A1) -> Net-(DRIVER6-B1)
- JM6 pad 3: Net-(DRIVER6-B1) -> Net-(DRIVER6-A2)
- JM6 pad 4: Net-(DRIVER6-A2) -> Net-(DRIVER6-B2)
- PS1 pad 1: Net-(PS1-+) -> GND
- PS1 pad 2: Net-(PS1--) -> Net-(PS1-+)
- TP4 pad 1: Net-(PS1--) -> GND
- U1 pad 16: CS_MOT_SPI_10 -> Net-(U1-PA2)
- U14 pad 1: UARTTX_MOT_U1 -> UARTTX_MOT
- U18 pad 2: +3V3 -> VMCU
- U19 pad 2: +3V3 -> VMCU
- U20 pad 2: +3V3 -> VMCU
- U21 pad 2: +3V3 -> VMCU
- U22 pad 2: +3V3 -> VMCU
- U6 pad 2: +3V3 -> VMCU
Routing:
- net UARTTX_MOT: track 0.00 -> 177.5 mm, vias 0 -> 6
- net STEP_MOT_U_10: track 0.00 -> 168.2 mm, vias 0 -> 2
- net DIAG_MOT_SPI_10: track 0.00 -> 156.5 mm, vias 0 -> 6
- net EN_MOT_U_10: track 0.00 -> 152.9 mm, vias 0 -> 3
- net DIR_MOT_U_10: track 0.00 -> 146.2 mm, vias 0 -> 4
- net EN_MOT_U_00: track 0.00 -> 132.6 mm, vias 0 -> 2
- net STEP_MOT_SPI_10: track 0.00 -> 125.9 mm, vias 0 -> 4
- net EN_MOT_SPI_10: track 0.00 -> 125.7 mm, vias 0 -> 3
- net SPI1_MISO: track 6.29 -> 123.4 mm, vias 1 -> 6
- net SPI1_MOSI: track 5.30 -> 118.7 mm, vias 1 -> 4
- net STEP_MOT_U_00: track 0.00 -> 112.0 mm, vias 0 -> 2
- net DIR_MOT_SPI_10: track 0.00 -> 112.0 mm, vias 0 -> 4
- net VMCU: track 83.9 -> 194.7 mm, vias 1 -> 36
- net SPI1_SCK: track 5.56 -> 115.5 mm, vias 1 -> 4
- net EN_MOT_U_01: track 0.00 -> 103.2 mm, vias 0 -> 2
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- added copper zone on F.Cu, net +24V
- added copper zone on F.Cu, net +5V
- added copper zone on In1.Cu, net GND
- added copper zone on F.Cu, net Net-(D1-K)
- added copper zone on F.Cu, net Net-(PS1-+)
- added copper zone on F.Cu, net VMCU
- added copper zone on In2.Cu, net VMCU
Other:
- board outline added: 163 x 83 mm
- board text added: "15A"
- board text added: "2209"
- board text added: "3.3V"
- board text added: "5160"
- board text added: "Arsenal's Motor Controller Board"
- board text added: "BOOT"
- board text added: "CAN_H"
- board text added: "CAN_L"
- board text added: "CLK"
- board text added: "CSN"
- board text added: "DIO"
- board text added: "Designed & routed by Atharva Chauhan · 2026 github.com/shadedvox/arsenal JLCPCB 4-layer, ENIG"
- board text added: "GND"
- board text added: "MCU: STM32F446RET6 (LQFP64) Interfaces: SPI x2 (Motor Drivers + Encoders) UART x3 (Motor Drivers + RPi) CAN BUS x1, PORTS x3 I2C BUS x1, PORTS x8 USB x1 SWD x1 Power: 24V Input, 5V + 3.3V Logic rails Supports 6 Motor and Encoder pairs."
- board text added: "MISO"
- board text added: "MOSI"
- board text added: "NRST"
- board text added: "PANDA WAS HERE"
- board text added: "RPI"
- board text added: "RX"
- board text added: "SCK"
- board text added: "SCL"
- board text added: "SDA"
- board text added: "SUPER SAIYAN"
- board text added: "SWD"
- board text added: "TX"
- board text added: "Throughout Heaven and Earth, I alone am the Honored One."
- board text added: "VOXBOARD v1.0"
- board text added: "vox"

Commit message: Major Update
Parts:
- moved G*** 0.40 mm to (129.6, 39.8)
Routing:
- net NRST: track 39.0 -> 39.7 mm
Other:
- board text added: "Eight-Handled Sword Divergent Sila Divine General Mahoraga"

Commit message: Updates
Parts:
- C24: footprint Capacitor_THT:CP_Radial_D8.0mm_P3.50mm -> Capacitor_THT:CP_Radial_D12.5mm_P5.00mm
- C25, C29, C58, C7: footprint Capacitor_SMD:C_0603_1608Metric -> Capacitor_SMD:C_0805_2012Metric
- C53: footprint Capacitor_THT:CP_Radial_D8.0mm_P3.50mm -> Capacitor_THT:CP_Radial_D6.3mm_P2.50mm
- D2: footprint Diode_SMD:D_SMA -> Diode_SMD:D_SMC
- D8: footprint Diode_SMD:D_SMC -> Package_TO_SOT_SMD:SOT-23
- R2: footprint Resistor_SMD:R_0402_1005Metric -> Resistor_SMD:R_0603_1608Metric
- moved TP6 8.50 mm to (97.2, 62.0), turned to 180 degrees
- moved TP5 7.64 mm to (109.0, 59.4)
- moved R5 6.24 mm to (92.3, 64.1), turned to 0 degrees
- moved D2 3.86 mm to (112.6, 64.4), turned to 0 degrees
- moved D1 3.75 mm to (151.7, 53.1)
- moved R8 3.75 mm to (152.2, 50.2)
- moved D8 2.79 mm to (95.1, 58.4)
- moved Q2 2.55 mm to (145.8, 54.2)
- moved D3 2.47 mm to (91.5, 62.7), turned to 0 degrees
- moved C15 1.84 mm to (115.4, 49.1)
- moved C21 1.42 mm to (92.5, 58.1)
- moved R2 1.29 mm to (112.2, 49.0), turned to 0 degrees
- moved C16 1.11 mm to (108.9, 49.0)
- moved C20 1.08 mm to (109.2, 56.8)
- moved IC1 1.08 mm to (111.1, 52.8)
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Routing:
- net +24V: track 20.5 -> 30.5 mm
- net Net-(D2-K): track 9.40 -> 14.5 mm
- net Net-(D1-A): track 6.81 -> 9.48 mm
- net Net-(IC1-COMP): track 5.75 -> 3.38 mm
- net Net-(D5-A): track 36.0 -> 37.3 mm
- net Net-(D3-K): track 1.39 -> 2.43 mm
- net +5V: track 8.98 -> 8.00 mm
- net VMCU: track 194.7 -> 194.1 mm
- net GND: track 321.2 -> 321.7 mm, vias 94 -> 95
- net Net-(PS1-+): track 11.6 -> 12.2 mm

Commit message: Updated JOURNAL.md
Routing:
- net GND: track 321.7 -> 288.8 mm, vias 95 -> 1669
- net Net-(IC1-COMP): track 3.38 -> 5.74 mm
- net STEP_MOT_U_10: vias 2 -> 3
- added copper zone on B.Cu, net GND
- added copper zone on F.Cu, net GND
