File: Stage1 - STM/voxboard/voxboard-backups/voxboard-2026-07-28_005139/voxboard.kicad_sch (KiCad schematic)
At the start: 179 parts, among them IC1 TPS54331DR, J1 USB4110-GF-A, J11 Conn_01x04_Pin, J12 Conn_01x04_Pin, J13 Conn_01x04_Pin, J14 Conn_01x04_Pin, J15 Conn_01x04_Pin, J16 Conn_01x04_Pin, J17 Conn_01x04_Pin, J18 Conn_01x04_Pin, Q1 PMOS, Q2 PMOS, SW2 SW_Push, SW3 SW_SPDT, U1 STM32F446RETx, U11 SN65HVD230DR, U12 TPD4E02B04DQAR, U14 PESD5V0F1BRSFYL, U16 SM12OC, U18 MT6835, U19 MT6835, U2 AP7361C-33Y5-13, U20 MT6835, U21 MT6835, U22 MT6835, U3 TPD4E02B04DQAR, U4 SM12OC, U5 TPD2E1B06DRLR, U6 MT6835, Y1 8MHz

Commit message: Bulk
Parts:
- removed C49: 100n, Capacitor_SMD:C_0402_1005Metric, symbol Device:C
- removed C50: 1u, Capacitor_SMD:C_0603_1608Metric, symbol Device:C
- removed C51: 22u, Capacitor_THT:CP_Radial_D5.0mm_P2.00mm, symbol Device:C_Polarized
- removed C58: 10u, Capacitor_SMD:C_0603_1608Metric, symbol Device:C
- added FB1: 600R, Inductor_SMD:L_1210_3225Metric, symbol Device:FerriteBead
- JM1, JM2, JM3, JM4, JM5, JM6: footprint Connector_JST:JST_XA_B04B-XASK-1_1x04_P2.50mm_Vertical -> Arsenal_Lib:JST_VH_B4P-VH-FB-B_1x04_P3.96mm_Vertical
Connections:
- net +3.3V: no longer U18.2 (VDD), U19.2 (VDD), U20.2 (VDD), U21.2 (VDD), U22.2 (VDD), U6.2 (VDD)
- net GND: now also FB1.2; no longer PS1.1 (-), TP4.1
- net at F1.1: now also PS1.1 (+); no longer PS1.2 (+)
- net at JM5.1 (Pin_1): now also DRIVER5.4 (B2); no longer DRIVER5.5 (A1)
- net at JM5.2 (Pin_2): now also DRIVER5.5 (A1); no longer DRIVER5.3 (B1)
- net at JM5.3 (Pin_3): now also DRIVER5.3 (B1); no longer DRIVER5.6 (A2)
- net at JM5.4 (Pin_4): now also DRIVER5.6 (A2); no longer DRIVER5.4 (B2)
- net at DRIVER4.3 (B1): now also JM4.3 (Pin_3); no longer JM4.2 (Pin_2)
- net at DRIVER4.4 (B2): now also JM4.1 (Pin_1); no longer JM4.4 (Pin_4)
- net at DRIVER4.5 (A1): now also JM4.2 (Pin_2); no longer JM4.1 (Pin_1)
- net at DRIVER4.6 (A2): now also JM4.4 (Pin_4); no longer JM4.3 (Pin_3)
- net at JM6.1 (Pin_1): now also DRIVER6.4 (B2); no longer DRIVER6.5 (A1)
- net at JM6.2 (Pin_2): now also DRIVER6.5 (A1); no longer DRIVER6.3 (B1)
- net at JM6.3 (Pin_3): now also DRIVER6.3 (B1); no longer DRIVER6.6 (A2)
- net at JM6.4 (Pin_4): now also DRIVER6.6 (A2); no longer DRIVER6.4 (B2)
- net at DRIVER3.4 (B1): now also JM3.1 (Pin_1); no longer JM3.2 (Pin_2)
- net at DRIVER3.5 (A1): now also JM3.2 (Pin_2); no longer JM3.1 (Pin_1)
- net at DRIVER1.4 (B1): now also JM1.1 (Pin_1); no longer JM1.2 (Pin_2)
- net at DRIVER1.5 (A1): now also JM1.2 (Pin_2); no longer JM1.1 (Pin_1)
- net at JM2.1 (Pin_1): now also DRIVER2.4 (B1); no longer DRIVER2.5 (A1)
- net at JM2.2 (Pin_2): now also DRIVER2.5 (A1); no longer DRIVER2.4 (B1)
- new net: FB1.1, PS1.2 (-), TP4.1
- new net +3V3: U18.2 (VDD), U19.2 (VDD), U20.2 (VDD), U21.2 (VDD), U22.2 (VDD), U6.2 (VDD)
Other:
- title: Arsenal - VoxBoard - Schematics -> Arsenal - Main Board
- moved on the sheet: JM4
